File: Beacon/Wiring/BeaconWiringSchematic/BeaconWiringSchematic.sch (KiCad schematic (older format))
At the start: 22 parts, among them J1 Header Pin, J2 Header Pin, SW1 SW_Push, SW2 SW_DIP_x01, U1 GPS, U2 TTLAdaptor, U3 Charger, U4 MPU6050, U5 MCP1826S, U6 ESP32

Commit message: Added typescript version of beacon code to beacon folder
Parts:
- added J? (x2): Header Pin, symbol Connector:Conn_01x01_Male
- U6: symbol maenford_components:ESP32 -> BeaconWiringSchematic-rescue:ESP32-maenford_components
Connections:
- net +3V3: now also J?.1 (Pin_1); no longer U1.1 (VCC), U4.1 (VCC)
- net Rx: now also U6.3 (U0T); no longer U6.2 (U0R)
- net Tx: now also U6.2 (U0R); no longer U6.3 (U0T)
- net at R4.2: now also U6.16 (GPIO4); no longer U6.12 (GPIO13)
- net ADC2_CH1 renamed ADC
- net ADC: now also U6.12 (GPIO13); no longer U6.16 (GPIO4)
- new net VCC: J?.1 (Pin_1), U1.1 (VCC), U4.1 (VCC)
Changed lines of the file:
@@
 EESchema Schematic File Version 4
+LIBS:BeaconWiringSchematic-cache
 EELAYER 29 0
 EELAYER END
@@
 $EndDescr
 $Comp
-L maenford_components:ESP32 U6
+L BeaconWiringSchematic-rescue:ESP32-maenford_components U6
 U 1 1 5EA88EC5
 P 2950 2600
@@
 	2350 1850 2050 1850
 Text Label 2050 1750 2    50   ~ 0
+Tx
+Text Label 2050 1850 2    50   ~ 0
 Rx
-Text Label 2050 1850 2    50   ~ 0
-Tx
 Text Label 1100 1000 0    50   ~ 0
 Rx
@@
 $EndComp
 $Comp
-L power:+3.3V #PWR015
-U 1 1 5EABBC12
-P 2350 2350
-F 0 "#PWR015" H 2350 2200 50  0001 C CNN
-F 1 "+3.3V" V 2365 2478 50  0000 L CNN
-F 2 "" H 2350 2350 50  0001 C CNN
-F 3 "" H 2350 2350 50  0001 C CNN
-	1    2350 2350
-	0    -1   -1   0
-$EndComp
-$Comp
 L power:+3.3V #PWR018
 U 1 1 5EABC3FE
@@
 	4000 4600 3900 4600
 $Comp
-L power:+3.3V #PWR011
-U 1 1 5EACD8C5
-P 1950 650
-F 0 "#PWR011" H 1950 500 50  0001 C CNN
-F 1 "+3.3V" V 1965 778 50  0000 L CNN
-F 2 "" H 1950 650 50  0001 C CNN
-F 3 "" H 1950 650 50  0001 C CNN
-	1    1950 650
-	0    -1   -1   0
-$EndComp
-$Comp
-L power:+3.3V #PWR02
-U 1 1 5EACE28D
-P 1100 1100
-F 0 "#PWR02" H 1100 950 50  0001 C CNN
-F 1 "+3.3V" V 1115 1228 50  0000 L CNN
-F 2 "" H 1100 1100 50  0001 C CNN
-F 3 "" H 1100 1100 50  0001 C CNN
-	1    1100 1100
-	0    1    1    0
-$EndComp
-$Comp
 L Connector:Conn_01x01_Male J2
 U 1 1 5EAD98B8
@@
 $EndComp
 NoConn ~ 2350 1950
-Text Label 3550 1650 0    50   ~ 0
-ADC2_CH1
 Text Label 3600 4250 0    50   ~ 0
-ADC2_CH1
+ADC
 Text Label 3550 1750 0    50   ~ 0
 SCL
@@
 Wire Wire Line
 	4150 2150 3550 2150
-Wire Wire Line
-	3550 2050 4150 2050
-Wire Wire Line
-	4150 2050 4150 1800
 $Comp
 L Regulator_Linear:MCP1826S U5
@@
 	0    -1   -1   0
 $EndComp
+$Comp
+L power:VCC #PWR?
+U 1 1 5EADDAF8
+P 1100 1100
+F 0 "#PWR?" H 1100 950 50  0001 C CNN
+F 1 "VCC" V 1117 1228 50  0000 L CNN
+F 2 "" H 1100 1100 50  0001 C CNN
+F 3 "" H 1100 1100 50  0001 C CNN
+	1    1100 1100
+	0    1    1    0
+$EndComp
+$Comp
+L power:VCC #PWR?
+U 1 1 5EADE699
+P 1950 650
+F 0 "#PWR?" H 1950 500 50  0001 C CNN
+F 1 "VCC" V 1968 777 50  0000 L CNN
+F 2 "" H 1950 650 50  0001 C CNN
+F 3 "" H 1950 650 50  0001 C CNN
+	1    1950 650
+	0    -1   -1   0
+$EndComp
+$Comp
+L power:VCC #PWR?
+U 1 1 5EADF293
+P 2750 2900
+F 0 "#PWR?" H 2750 2750 50  0001 C CNN
+F 1 "VCC" V 2767 3028 50  0000 L CNN
+F 2 "" H 2750 2900 50  0001 C CNN
+F 3 "" H 2750 2900 50  0001 C CNN
+	1    2750 2900
+	0    1    1    0
+$EndComp
+$Comp
+L Connector:Conn_01x01_Male J?
+U 1 1 5EAE0B69
+P 2550 2900
+F 0 "J?" H 2658 3081 50  0000 C CNN
+F 1 "Header Pin" H 2658 2990 50  0000 C CNN
+F 2 "" H 2550 2900 50  0001 C CNN
+F 3 "~" H 2550 2900 50  0001 C CNN
+	1    2550 2900
+	1    0    0    -1
+$EndComp
+$Comp
+L Connector:Conn_01x01_Male J?
+U 1 1 5EAE1404
+P 2550 2700
+F 0 "J?" H 2658 2881 50  0000 C CNN
+F 1 "Header Pin" H 2658 2790 50  0000 C CNN
+F 2 "" H 2550 2700 50  0001 C CNN
+F 3 "~" H 2550 2700 50  0001 C CNN
+	1    2550 2700
+	1    0    0    -1
+$EndComp
+Wire Wire Line
+	4150 1800 4150 1650
+Wire Wire Line
+	4150 1650 3550 1650
+Text Label 3550 2050 0    50   ~ 0
+ADC
+$Comp
+L power:+3.3V #PWR?
+U 1 1 5EAE5915
+P 2350 2350
+F 0 "#PWR?" H 2350 2200 50  0001 C CNN
+F 1 "+3.3V" H 2365 2523 50  0000 C CNN
+F 2 "" H 2350 2350 50  0001 C CNN
+F 3 "" H 2350 2350 50  0001 C CNN
+	1    2350 2350
+	0    -1   -1   0
+$EndComp
+$Comp
+L power:+3.3V #PWR?
+U 1 1 5EAE628F
+P 2750 2700
+F 0 "#PWR?" H 2750 2550 50  0001 C CNN
+F 1 "+3.3V" H 2765 2873 50  0000 C CNN
+F 2 "" H 2750 2700 50  0001 C CNN
+F 3 "" H 2750 2700 50  0001 C CNN
+	1    2750 2700
+	0    1    1    0
+$EndComp
 $EndSCHEMATC
